File: pcb/epaper-smart-watch.kicad_pcb (KiCad board)
At the start: 4 copper layers, 41.6 x 36 mm, 101 parts, among them IC2 NPM1100-QDAA-R7, IC3 MAX17048G+T10, IC4 AP3032, J16 Touch3, J17 Touch2, J18 Touch1, J5 Lithium Battery 3.7V, J6 AXT624124, M1 Motor_DC, P1 USB_C_Plug_USB2.0, Q2 Si1308EDL, Q3 AO3400A, Q4 AO3400A, SW2 BTN, SW3 BTN, SW4 BTN, SW5 BTN, SW6 SW_Push, U1 BME280, U2 USBLC6-2SC6, U3 STM32WB5MMG, U4 XT25F32FDTIGT, U5 XC6206P332MR

Commit message: V2 design as sent to fabrication
- Swap 10k resistors (R1/R2/R16-R19) to JLCPCB basic part C25744
  (UNI-ROYAL) in the parts db, replacing extended FOJAN C2906861
- Regenerate gerbers and production files from the final board
- Add Panasonic AXT524124 24-pin FPC footprint and 3D model,
  remove the old AXT624124 footprint
- Remove auto-layout tooling and the coopt-routed board variant
- Ignore KiCad DRC/ERC .rpt report files

Pre-order verification: ERC/DRC clean (warnings all cosmetic/known),
0 unconnected, 0 schematic-parity issues; sch/board/BOM/CPL/parts-db
cross-check clean; inductors verified against nPM1100, EPD boost
reference, and AP3032 requirements.

Co-Authored-By: Claude Fable 5 <noreply@anthropic.com>
Parts:
- added C28: 100nF/16V, Capacitor_SMD:C_0402_1005Metric, F.Cu at (158.8, 90.1)
- C10: value 0.1uF -> 100nF/16V
- C11, C24, C25, C26, C6: value 100nF -> 100nF/16V
- C12: value 0.1uF/6.3V -> 100nF/16V
- C13: value 10uF/6.3V -> 10uF/10V
- C14, C19, C20: value 1uF/25V -> 1uF/50V
- C16: value 1uF/16V -> 1uF/50V
- C18, C27, C5: value 1uF/16V -> 1uF/25V
- C2, C22, C3, C4: value 10uF -> 10uF/10V
- C8: value 1uF -> 1uF/25V
- C9: value 0.1uF/16V -> 100nF/16V
- D1, D2, D3: value LED -> LED White
- J6: value AXT624124 -> AXT524124; footprint ProjectLibrary:AXT624124 -> ProjectLibrary:PANASONIC_AXT524124
- LS1: value CPT-9019S-SMT-TR -> CPT-9019B-SMT-TR
- R10: footprint Resistor_SMD:R_0402_1005Metric -> Resistor_SMD:R_0603_1608Metric
- SW2, SW3, SW4, SW5: footprint Button_Switch_SMD:SW_SPST_B3U-3000P-B -> Button_Switch_SMD:SW_SPST_B3U-3000P
- moved C19 11.2 mm to (136.7, 97.0), turned to 90 degrees
- moved J11 4.50 mm to (133.9, 99.6)
- moved C16 3.46 mm to (145.8, 110.4)
- moved R13 3.04 mm to (153.0, 100.3), turned to 0 degrees
- moved R10 2.91 mm to (146.9, 107.0)
- moved J4 2.72 mm to (155.7, 100.4)
- moved C18 2.44 mm to (138.2, 95.0), turned to 0 degrees
- moved L3 2.38 mm to (146.2, 104.7), turned to 0 degrees
- moved R9 2.28 mm to (145.3, 102.6), turned to 180 degrees
- moved R20 1.75 mm to (147.2, 102.6), turned to 180 degrees
- moved R11 1.50 mm to (143.4, 110.3), turned to 180 degrees
- moved C12 1.30 mm to (134.4, 107.9)
- moved R5 1.22 mm to (153.5, 102.6), turned to 0 degrees
- moved C21 0.47 mm to (134.4, 97.7)
- moved J6 0.46 mm to (135.6, 102.4), turned to -90 degrees
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Routing:
- net /SND: track 42.7 -> 32.5 mm
- net Net-(P1-D--PadA7): track 4.51 -> 9.70 mm
- net /EPD_LIGHT_PWR_NEG: track 21.6 -> 16.7 mm
- net Net-(J6-Pin_5): track 10.2 -> 6.01 mm
- net Net-(J6-Pin_7): track 5.50 -> 9.49 mm, vias 0 -> 2
- net Net-(J6-Pin_19): track 8.89 -> 12.5 mm, vias 0 -> 2
- net +3V0: track 134.6 -> 137.9 mm, vias 14 -> 16
- net /EPD_BUSY: track 23.4 -> 25.3 mm
- net Net-(P1-CC1): track 1.55 -> 3.34 mm
- net /EPD_SPICL: track 29.8 -> 28.2 mm
- net Net-(IC2-ICHG): track 2.48 -> 1.11 mm
- net Net-(IC4-OV): track 4.17 -> 5.50 mm
- net /EPD_RESR: track 11.2 -> 9.89 mm
- net /EPD_LIGHT: track 25.7 -> 24.4 mm
- net /VSYS: track 67.6 -> 68.9 mm
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