File: pcb/epaper-smart-watch.kicad_sch (KiCad schematic)
At the start: 99 parts, among them IC2 NPM1100-QDAA-R7, IC3 MAX17048G+T10, IC4 AP3032, J16 Touch3, J17 Touch2, J18 Touch1, J5 Lithium Battery 3.7V, J6 AXT624124, M1 Motor_DC, P1 USB_C_Plug_USB2.0, Q2 Si1308EDL, Q3 AO3400A, Q4 AO3400A, SW2 BTN, SW3 BTN, SW4 BTN, SW5 BTN, SW6 SW_Push, U1 BME280, U2 USBLC6-2SC6, U3 STM32WB5MMG, U4 XT25F32FDTIGT, U5 XC6206P332MR

Commit message: V2 design as sent to fabrication
- Swap 10k resistors (R1/R2/R16-R19) to JLCPCB basic part C25744
  (UNI-ROYAL) in the parts db, replacing extended FOJAN C2906861
- Regenerate gerbers and production files from the final board
- Add Panasonic AXT524124 24-pin FPC footprint and 3D model,
  remove the old AXT624124 footprint
- Remove auto-layout tooling and the coopt-routed board variant
- Ignore KiCad DRC/ERC .rpt report files

Pre-order verification: ERC/DRC clean (warnings all cosmetic/known),
0 unconnected, 0 schematic-parity issues; sch/board/BOM/CPL/parts-db
cross-check clean; inductors verified against nPM1100, EPD boost
reference, and AP3032 requirements.

Co-Authored-By: Claude Fable 5 <noreply@anthropic.com>
Parts:
- added C28: 100nF/16V, Capacitor_SMD:C_0402_1005Metric, symbol Device:C_Small
- AC1: LCSC (none) -> C437655
- C10: value 0.1uF -> 100nF/16V; LCSC (none) -> C1525
- C11, C24, C25, C26, C6: value 100nF -> 100nF/16V; LCSC (none) -> C1525
- C12: value 0.1uF/6.3V -> 100nF/16V; LCSC (none) -> C1525
- C13: value 10uF/6.3V -> 10uF/10V; LCSC (none) -> C19702
- C14, C19, C20: value 1uF/25V -> 1uF/50V; LCSC (none) -> C15849
- C15, C23: LCSC (none) -> C28323
- C16: value 1uF/16V -> 1uF/50V; LCSC (none) -> C15849
- C17: LCSC (none) -> C1779
- C18, C27, C5: value 1uF/16V -> 1uF/25V; LCSC (none) -> C52923
- C2, C22, C3, C4: value 10uF -> 10uF/10V; LCSC (none) -> C19702
- C21: LCSC (none) -> C1623
- C7: LCSC (none) -> C377773
- C8: value 1uF -> 1uF/25V; LCSC (none) -> C52923
- C9: value 0.1uF/16V -> 100nF/16V; LCSC (none) -> C1525
- D1, D2, D3: value LED -> LED White; LCSC (none) -> C2290
- D5, D6, D7, D8, D9: LCSC (none) -> C77336
- IC2: LCSC (none) -> C7249859
- IC3: LCSC (none) -> C2682616
- IC4: LCSC (none) -> C264086
- J6: value AXT624124 -> AXT524124; footprint ProjectLibrary:AXT624124 -> ProjectLibrary:PANASONIC_AXT524124; LCSC (none) -> C2859266
- L1: LCSC (none) -> C394950
- L2: LCSC (none) -> C6364771
- L3: LCSC (none) -> C50325627
- LS1: value CPT-9019S-SMT-TR -> CPT-9019B-SMT-TR; LCSC (none) -> C18212234
- P1: LCSC (none) -> C2906290
- Q2: LCSC (none) -> C469327
- Q3, Q4: LCSC (none) -> C20917
- R1, R16, R17, R18, R19, R2: LCSC (none) -> C25744
- R10: footprint Resistor_SMD:R_0402_1005Metric -> Resistor_SMD:R_0603_1608Metric; LCSC (none) -> C23240
- R11, R12, R14, R20, R23, R8: LCSC (none) -> C25741
- R13, R21, R24, R6: LCSC (none) -> C11702
- R15, R22, R7: LCSC (none) -> C25076
- R3, R4: LCSC (none) -> C25905
- R5: LCSC (none) -> C25768
- R9: LCSC (none) -> C2090812
- SW2, SW3, SW4, SW5: footprint Button_Switch_SMD:SW_SPST_B3U-3000P-B -> Button_Switch_SMD:SW_SPST_B3U-3000P; LCSC (none) -> C963349
- SW6: LCSC (none) -> C720477
- SWD1: LCSC (none) -> C5306612; now left out of the parts list
- U1: LCSC (none) -> C92489
- U2: LCSC (none) -> C7519
- U3: LCSC (none) -> C5184586
- U4: LCSC (none) -> C7429719; LCSC Part C7429719 -> (none)
- U5: LCSC (none) -> C5446
Connections:
- net +3V0: now also C28.1
- net GND: now also C28.2
